File: ADSR/ADSR.kicad_pcb (KiCad board)
At the start: 2 copper layers, 45 x 52 mm, 24 parts, among them J1 INPUT, J2 NJ2FD-V, J3 NJ2FD-V, U1 TL074

Commit message: added the layout of the PCB ADSL
Parts:
- moved R1 8.38 mm to (159.1, 100.9), turned to 120 degrees
Routing:
- net Net-(U1C--): track 0.00 -> 31.2 mm
- net Net-(U1D-+): track 0.00 -> 29.6 mm, vias 0 -> 2
- net /Vin_minus: track 0.00 -> 25.4 mm, vias 0 -> 2
- net /Vin_plus: track 0.00 -> 23.1 mm
- net Net-(D5-K): track 0.00 -> 18.5 mm, vias 0 -> 2
- net Net-(D6-A): track 0.00 -> 16.5 mm
- net Net-(U1A--): track 0.00 -> 15.9 mm, vias 0 -> 2
- net Net-(U1C-+): track 0.00 -> 9.70 mm
- net Net-(D3-A): track 0.00 -> 9.04 mm
- net Net-(D3-K): track 0.00 -> 7.75 mm, vias 0 -> 1
- net Net-(D7-A): track 0.00 -> 7.10 mm, vias 0 -> 2
- net Net-(D5-A): track 0.00 -> 6.88 mm, vias 0 -> 2
- net Net-(D4-K): track 0.00 -> 5.71 mm
- net Net-(J3-PadT): track 0.00 -> 4.80 mm
- net Net-(D1-A): track 0.00 -> 4.19 mm
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- added copper zone on B.Cu, net 0
- added copper zone on F.Cu, net 0
- added copper zone on F.Cu, net Net-(D4-A)
Other:
- rule pad_to_mask_clearance: 0 -> 0.1
