File: sequencer/sequencer.kicad_sch (KiCad schematic)
At the start: 35 parts, among them J1 INPUT, J2 Conn_01x06_Pin, J3 Conn_01x06_Pin, SW1 SW_DIP_x06, SW2 SW_DIP_x06, U1 TL074

Commit message: sch pasmix, mix
Parts:
- removed SW1: SW_DIP_x06, Button_Switch_SMD:SW_DIP_SPSTx06_Slide_9.78x17.42mm_W8.61mm_P2.54mm, symbol Switch:SW_DIP_x06
- added J?: Conn_01x06_Pin, Connector_PinHeader_2.54mm:PinHeader_1x06_P2.54mm_Vertical, symbol Connector:Conn_01x06_Pin
Connections:
- net RES: now also J?.1 (Pin_1)
- net S3: now also J?.2 (Pin_2)
- net S4: now also J?.3 (Pin_3)
- net S5: now also J?.4 (Pin_4)
- net S6: now also J?.5 (Pin_5)
- new net S7: J?.6 (Pin_6)
Other:
- note added: "Connections to the mix/pot"
- note added: "For Looping (Connect the RES, Pin1, to one of the other pins)"
- note added: "the mixer that I created was just a mixer, not useful for this part. For the sequencer we need a dupong 6 pin input that will be connected to the sequencer board 6 duponts. This other board will be half hexagon i guess and it has to contain the 6 potentiometers. Potentially could be even another hexagon since we saw that it fits to have 6 hexagones there and it has as output directly the CV at th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"
- note removed: "Switch for the reset. Please select JUST ONE Sostituiisci con i conn 01x07 e il 07 corrisponde al reset"
- moved on the sheet: J2
